File: inky-esp32-carrier/inky-esp32-carrier.kicad_sch (KiCad schematic)
At the start: 29 parts, among them J1 USB_C_Receptacle, J2 Inky_Impression_GPIO, J3 UART0, SW1 RESET, SW2 BOOT, U1 ESP32-S3-WROOM-1-N16R8, U2 SGM2212-3.3XKC3G/TR

Commit message: Setup page: restart the frame after saving or drawing
Taking the serial port stops the frame's loop, so saving settings or drawing a
block left the frame idle until someone reset it by hand. Both now reset the
board when they finish.

Co-Authored-By: Claude Opus 5 <noreply@anthropic.com>
Parts:
- removed H3, H4: MountingHole_M2.5, MountingHole:MountingHole_2.7mm_M2.5, symbol Mechanical:MountingHole
Changed lines of the file:
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@@
   (property "Description" "" (at 243.84 226.06 0) (effects (font (size 1.27 1.27))) (hide yes))
   (instances (project "inky-esp32-carrier" (path "/55b3ea2b-612e-4a33-9791-ff6f3419debb" (reference "H2") (unit 1)))))
-(symbol (lib_id "Mechanical:MountingHole") (at 266.70 226.06 0) (unit 1) (exclude_from_sim no) (in_bom no) (on_board yes) (dnp no)
-  (property "Reference" "H3" (at 266.70 222.25 0) (effects (font (size 1.27 1.27))))
-  (property "Value" "MountingHole_M2.5" (at 266.70 229.87 0) (effects (font (size 1.27 1.27))))
-  (property "Footprint" "MountingHole:MountingHole_2.7mm_M2.5" (at 266.70 226.06 0) (effects (font (size 1.27 1.27))) (hide yes))
-  (property "Datasheet" "" (at 266.70 226.06 0) (effects (font (size 1.27 1.27))) (hide yes))
-  (property "Description" "" (at 266.70 226.06 0) (effects (font (size 1.27 1.27))) (hide yes))
-  (instances (project "inky-esp32-carrier" (path "/55b3ea2b-612e-4a33-9791-ff6f3419debb" (reference "H3") (unit 1)))))
-(symbol (lib_id "Mechanical:MountingHole") (at 289.56 226.06 0) (unit 1) (exclude_from_sim no) (in_bom no) (on_board yes) (dnp no)
-  (property "Reference" "H4" (at 289.56 222.25 0) (effects (font (size 1.27 1.27))))
-  (property "Value" "MountingHole_M2.5" (at 289.56 229.87 0) (effects (font (size 1.27 1.27))))
-  (property "Footprint" "MountingHole:MountingHole_2.7mm_M2.5" (at 289.56 226.06 0) (effects (font (size 1.27 1.27))) (hide yes))
-  (property "Datasheet" "" (at 289.56 226.06 0) (effects (font (size 1.27 1.27))) (hide yes))
-  (property "Description" "" (at 289.56 226.06 0) (effects (font (size 1.27 1.27))) (hide yes))
-  (instances (project "inky-esp32-carrier" (path "/55b3ea2b-612e-4a33-9791-ff6f3419debb" (reference "H4") (unit 1)))))
 (sheet_instances (path "/" (page "1")))
 (embedded_fonts no)
